File: midea_dongle.kicad_pcb (KiCad board)
At the start: 4 copper layers, 20 x 41.9 mm, 28 parts, among them J1 USB_A, J2 USB_C_Receptacle_USB2.0_14P, J3 Conn_01x02_Pin, J4 Conn_01x02_Pin, SW1 SW_Push, SW2 SW_Push, U1 SP3485EN, U2 AP2112K-3.3, U3 ESP32-C6-WROOM-1, U4 TXS0102DCT

Commit message: 5V bypass cap, correct button silk
Parts:
- added C6: 100n, Capacitor_SMD:C_0402_1005Metric, F.Cu at (126.0, 109.8)
- moved C4 0.25 mm to (128.8, 107.5)
Connections:
- net /BOOT renamed /USER_BTN
Routing:
- net /+5V_UART: track 6.43 -> 8.96 mm
- net +3.3V: track 73.1 -> 72.4 mm
- net GND: track 32.2 -> 32.8 mm, vias 21 -> 22
- net Net-(D1-K): track 15.0 -> 14.5 mm
Other:
- board text added: "Midea Matter Dongle REV 2.0"
- board text added: "RST"
- board text added: "USER"
- board text removed: "BOOT"
- board text removed: "COMM"
- board text removed: "Midea Matter Dongle REV 1.0"
