File: midea_dongle.kicad_sch (KiCad schematic)
At the start: 28 parts, among them J1 USB_A, J2 USB_C_Receptacle_USB2.0_14P, J3 Conn_01x02_Pin, J4 Conn_01x02_Pin, SW1 SW_Push, SW2 SW_Push, U1 SP3485EN, U2 AP2112K-3.3, U3 ESP32-C6-WROOM-1, U4 TXS0102DCT

Commit message: 5V bypass cap, correct button silk
Parts:
- added C6: 100n, Capacitor_SMD:C_0402_1005Metric, symbol Device:C
Connections:
- net +5V_UART: now also C6.1
- net GND: now also C6.2
- net BOOT renamed USER_BTN
Other:
- moved on the sheet: C5
